File: LM2596project.kicad_sch (KiCad schematic)
At the start: 11 parts, among them J1 Screw_Terminal_01x02, J2 Screw_Terminal_01x02, U1 LM2596S-ADJ

Commit message: Add files via upload
Other:
- moved on the sheet: J1, J2
Changed lines of the file:
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@@
+	)
+	(junction
+		(at 16.51 -24.384)
+		(diameter 0)
+		(color 0 0 0 0)
+	)
+	(junction
+		(at 41.656 -6.604)
+		(diameter 0)
+		(color 0 0 0 0)
 	)
 	(junction
@@
 	)
 	(junction
-		(at 16.51 -24.384)
-		(diameter 0)
-		(color 0 0 0 0)
-	)
-	(junction
-		(at 41.656 -6.604)
-		(diameter 0)
-		(color 0 0 0 0)
-	)
-	(junction
 		(at -34.544 -11.684)
 		(diameter 0)
@@
 	(wire
 		(pts
-			(xy 57.15 -6.604) (xy 81.534 -6.604)
-		)
-		(stroke
-			(width 0)
-			(type default)
-		)
-	)
-	(wire
-		(pts
-			(xy 84.074 -15.494) (xy 84.074 29.21)
+			(xy 57.15 -6.604) (xy 79.502 -6.604)
 		)
 		(stroke
@@
 	(wire
 		(pts
+			(xy -50.8 -11.684) (xy -34.544 -11.684)
+		)
+		(stroke
+			(width 0)
+			(type default)
+		)
+	)
+	(wire
+		(pts
 			(xy 41.656 -6.604) (xy 57.15 -6.604)
 		)
@@
 	(wire
 		(pts
-			(xy -83.82 -11.684) (xy -50.8 -11.684)
-		)
-		(stroke
-			(width 0)
-			(type default)
-		)
-	)
-	(wire
-		(pts
-			(xy 81.534 -15.494) (xy 81.534 -6.604)
-		)
-		(stroke
-			(width 0)
-			(type default)
-		)
-	)
-	(wire
-		(pts
 			(xy 16.51 -6.604) (xy 16.51 8.128)
 		)
@@
 	(wire
 		(pts
+			(xy 79.502 -4.064) (xy 79.502 29.464)
+		)
+		(stroke
+			(width 0)
+			(type default)
+		)
+	)
+	(wire
+		(pts
+			(xy -81.28 -11.684) (xy -50.8 -11.684)
+		)
+		(stroke
+			(width 0)
+			(type default)
+		)
+	)
+	(wire
+		(pts
 			(xy 57.15 15.24) (xy 57.15 29.21)
 		)
@@
 	(wire
 		(pts
-			(xy -81.28 -15.494) (xy -81.28 29.21)
-		)
-		(stroke
-			(width 0)
-			(type default)
-		)
-	)
-	(wire
-		(pts
-			(xy -83.82 -15.494) (xy -83.82 -11.684)
-		)
-		(stroke
-			(width 0)
-			(type default)
-		)
-	)
-	(wire
-		(pts
 			(xy 16.51 -32.004) (xy 31.75 -32.004)
 		)
@@
 	(wire
 		(pts
-			(xy -50.8 -11.684) (xy -34.544 -11.684)
-		)
-		(stroke
-			(width 0)
-			(type default)
-		)
-	)
-	(wire
-		(pts
 			(xy -64.77 -24.384) (xy -64.77 29.21)
 		)
@@
 		(pts
 			(xy 57.15 -6.604) (xy 57.15 7.62)
+		)
+		(stroke
+			(width 0)
+			(type default)
+		)
+	)
+	(wire
+		(pts
+			(xy -81.28 -9.144) (xy -81.28 29.21)
 		)
 		(stroke
@@
 	(symbol
 		(lib_id "Connector:Screw_Terminal_01x02")
-		(at 81.534 -20.574 90)
+		(at 84.582 -6.604 0)
 		(unit 1)
 		(body_style 1)
@@
 		(dnp no)
 		(property "Reference" "J2"
-			(at 82.042 -25.146 90)
+			(at 89.154 -6.096 90)
 			(show_name no)
 			(do_not_autoplace no)
@@
 		)
 		(property "Value" "Screw_Terminal_01x02"
-			(at 75.184 -23.114 90)
+			(at 87.122 -12.954 90)
 			(show_name no)
 			(do_not_autoplace no)
@@
 		)
 		(property "Footprint" "TerminalBlock_Phoenix:TerminalBlock_Phoenix_PT-1,5-2-3.5-H_1x02_P3.50mm_Horizontal"
-			(at 81.534 -20.574 0)
+			(at 84.582 -6.604 0)
 			(hide yes)
 			(show_name no)
@@
 		)
 		(property "Datasheet" ""
-			(at 81.534 -20.574 0)
+			(at 84.582 -6.604 0)
 			(hide yes)
 			(show_name no)
@@
 		)
 		(property "Description" "Generic screw terminal, single row, 01x02, script generated (kicad-library-utils/schlib/autogen/connector/)"
-			(at 81.534 -20.574 0)
+			(at 84.582 -6.604 0)
 			(hide yes)
 			(show_name no)
@@
 	(symbol
 		(lib_id "Connector:Screw_Terminal_01x02")
-		(at -83.82 -20.574 90)
+		(at -86.36 -11.684 0)
+		(mirror y)
 		(unit 1)
 		(body_style 1)
@@
 		(dnp no)
 		(property "Reference" "J1"
-			(at -83.058 -25.146 90)
+			(at -87.122 -16.256 0)
 			(show_name no)
 			(do_not_autoplace no)
@@
 		)
 		(property "Value" "Screw_Terminal_01x02"
-			(at -90.678 -23.114 90)
+			(at -94.996 -14.478 0)
 			(show_name no)
 			(do_not_autoplace no)
@@
 		)
 		(property "Footprint" "TerminalBlock_Phoenix:TerminalBlock_Phoenix_PT-1,5-2-3.5-H_1x02_P3.50mm_Horizontal"
-			(at -83.82 -20.574 0)
+			(at -86.36 -11.684 0)
 			(hide yes)
 			(show_name no)
@@
 		)
 		(property "Datasheet" ""
-			(at -83.82 -20.574 0)
+			(at -86.36 -11.684 0)
 			(hide yes)
 			(show_name no)
@@
 		)
 		(property "Description" "Generic screw terminal, single row, 01x02, script generated (kicad-library-utils/schlib/autogen/connector/)"
-			(at -83.82 -20.574 0)
+			(at -86.36 -11.684 0)
 			(hide yes)
 			(show_name no)
@@
 	(symbol
 		(lib_id "power:GND")
-		(at 84.074 29.21 0)
+		(at 79.502 29.464 0)
 		(unit 1)
 		(body_style 1)
@@
 		(fields_autoplaced yes)
 		(property "Reference" "#PWR010"
-			(at 84.074 35.56 0)
+			(at 79.502 35.814 0)
 			(hide yes)
 			(show_name no)
@@
 		)
 		(property "Value" "GND"
-			(at 84.074 33.782 0)
+			(at 79.502 34.036 0)
 			(show_name no)
 			(do_not_autoplace no)
@@
 		)
 		(property "Footprint" ""
-			(at 84.074 29.21 0)
+			(at 79.502 29.464 0)
 			(hide yes)
 			(show_name no)
@@
 		)
 		(property "Datasheet" ""
-			(at 84.074 29.21 0)
+			(at 79.502 29.464 0)
 			(hide yes)
 			(show_name no)
@@
 		)
 		(property "Description" "Power symbol creates a global label with name \"GND\" , ground"
-			(at 84.074 29.21 0)
-			(hide yes)
-			(show_name no)
+			(at 79.502 29.464 0)
+			(hide yes)
+			(show_name no)
