File: LM2596project.kicad_pcb (KiCad board)
At the start: 2 copper layers, 56.1 x 32.9 mm, 15 parts, among them J1 Screw_Terminal_01x02, J2 Screw_Terminal_01x02, U1 LM2596S-ADJ

Commit message: Add files via upload
Connections:
- U1 pad : (no net) -> GND
Routing:
- net GND: track 0.00 -> 5.62 mm, vias 42 -> 50
Other:
- board text added: "IN"
- board text added: "OUT"
Changed lines of the file:
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@@
 		(45 "User.4" user)
 		(63 "User.13" user "Mechanical 13")
-		(67 "User.15" user "Mechanical 15")
+		(67 "User.15" user "PlaceBySch")
 	)
 	(setup
@@
 			(outputformat 1)
 			(mirror no)
-			(drillshape 1)
+			(drillshape 0)
 			(scaleselection 1)
-			(outputdirectory "")
+			(outputdirectory "Fabrication Folders/")
 		)
 	)
@@
 		(tags "THT Terminal Block Phoenix PT-1,5-2-3.5-H pitch 3.5mm size 7x7.6mm drill 1.2mm pad 2.4mm")
 		(property "Reference" "J2"
-			(at 6.2992 0.9652 180)
+			(at 4.2926 -4.0894 270)
 			(layer "F.SilkS")
 			(effects
@@
 			)
 			(scale
-				(xyz 1 1 0.7188)
+				(xyz 1 1 0.71875)
 			)
 			(rotate
@@
 		)
 		(pad "" smd roundrect
+			(at -7.65 3.4 90)
+			(size 4.6 1.1)
+			(layers "F.Cu" "F.Mask" "F.Paste")
+			(roundrect_rratio 0.227273)
+			(net "GND")
+			(pinfunction "~{ON}/OFF_5")
+			(pintype "input")
+			(thermal_bridge_width 0)
+			(thermal_gap 0)
+		)
+		(pad "" smd roundrect
 			(at -0.925 -2.775 90)
 			(size 4.55 5.25)
@@
 			(pintype "input")
 		)
-		(pad "5" smd roundrect
-			(at -7.65 3.4 90)
-			(size 4.6 1.1)
-			(layers "F.Cu" "F.Mask" "F.Paste")
-			(roundrect_rratio 0.227273)
-			(net "GND")
-			(pinfunction "~{ON}/OFF_5")
-			(pintype "input")
-		)
 		(embedded_fonts no)
 		(model "${KICAD10_3DMODEL_DIR}/Package_TO_SOT_SMD.3dshapes/TO-263-5_TabPin3.step"
@@
 	)
 	(gr_text "+"
-		(at 26.7081 129.6162 0)
+		(at 23.9903 129.5146 0)
+		(layer "F.SilkS")
+		(effects
+			(font
+				(size 3 3)
+				(thickness 0.75)
+				(bold yes)
+			)
+			(justify left bottom)
+		)
+	)
+	(gr_text "OUT"
+		(at 68.4911 129.7178 0)
 		(layer "F.SilkS")
 		(effects
@@
 		)
 	)
+	(gr_text "IN"
+		(at 27.5971 130.0988 0)
+		(layer "F.SilkS")
+		(effects
+			(font
+				(face "Times New Roman")
+				(size 3 3)
+				(thickness 0.75)
+				(bold yes)
+			)
+			(justify left bottom)
+		)
+		(render_cache "IN" 0
+			(polygon
+				(pts
+					(xy 29.134181 129.518458) (xy 29.134181 129.5888) (xy 27.68118 129.5888) (xy 27.68118 129.518458)
+					(xy 27.773321 129.518458) (xy 27.886874 129.506411) (xy 27.968043 129.474311) (xy 28.013956 129.435817)
+					(xy 28.050109 129.373194) (xy 28.064961 129.302803) (xy 28.07264 129.10813) (xy 28.07264 127.290963)
+					(xy 28.065041 127.092123) (xy 28.050109 127.017472) (xy 28.017798 126.968008) (xy 27.958884 126.921668)
+					(xy 27.882718 126.891936) (xy 27.773321 126.880635) (xy 27.68118 126.880635) (xy 27.68118 126.810293)
+					(xy 29.134181 126.810293) (xy 29.134181 126.880635) (xy 29.04204 126.880635) (xy 28.928623 126.89267)
+					(xy 28.847318 126.924782) (xy 28.800984 126.963213) (xy 28.763237 127.025898) (xy 28.748385 127.096289)
+					(xy 28.740706 127.290963) (xy 28.740706 129.10813) (xy 28.748607 129.306964) (xy 28.764153 129.381804)
+					(xy 28.797295 129.431164) (xy 28.856477 129.477425) (xy 28.932643 129.507157) (xy 29.04204 129.518458)
+				)
+			)
+			(polygon
+				(pts
+					(xy 30.274856 126.810293) (xy 31.645791 128.517734) (xy 31.645791 127.337857) (xy 31.635309 127.168826)
+					(xy 31.609345 127.061121) (xy 31.573984 126.996406) (xy 31.499647 126.933631) (xy 31.39353 126.893699)
+					(xy 31.244073 126.880635) (xy 31.244073 126.810293) (xy 32.162181 126.810293) (xy 32.162181 126.880635)
+					(xy 32.001212 126.910301) (xy 31.92551 126.939619) (xy 31.873076 126.985543) (xy 31.831171 127.057589)
+					(xy 31.807759 127.154081) (xy 31.797466 127.337857) (xy 31.797466 129.647418) (xy 31.727857 129.647418)
+					(xy 29.848591 127.331996) (xy 29.848591 129.10813) (xy 29.863572 129.265145) (xy 29.901909 129.36852)
+					(xy 29.958134 129.434011) (xy 30.075449 129.497233) (xy 30.209277 129.518458) (xy 30.274856 129.518458)
+					(xy 30.274856 129.5888) (xy 29.28897 129.5888) (xy 29.28897 129.518458) (xy 29.439667 129.504567)
+					(xy 29.541741 129.471335) (xy 29.608623 129.423752) (xy 29.65505 129.355565) (xy 29.686724 129.254368)
+					(xy 29.698931 129.10813) (xy 29.698931 127.147714) (xy 29.63958 127.074625) (xy 29.549987 126.971889)
+					(xy 29.483692 126.921668) (xy 29.407664 126.8945) (xy 29.28897 126.880635) (xy 29.28897 126.810293)
+				)
+			)
+		)
+	)
+	(segment
+		(start 53.0987 133.5532)
+		(end 53.0987 136.344846)
+		(width 0.75)
+		(layer "F.Cu")
+		(net "GND")
+	)
+	(segment
+		(start 49.6987 133.5532)
+		(end 49.6987 136.369)
+		(width 0.75)
+		(layer "F.Cu")
+		(net "GND")
+	)
+	(segment
+		(start 49.6987 136.369)
+		(end 49.6951 136.3726)
+		(width 0.75)
+		(layer "F.Cu")
+		(net "GND")
+	)
+	(segment
+		(start 53.0987 136.344846)
+		(end 53.09605 136.347496)
+		(width 0.75)
+		(layer "F.Cu")
+		(net "GND")
+	)
 	(via
 		(at 67.9323 142.1892)
@@
 	)
 	(via
+		(at 45.8343 129.9972)
+		(size 0.6)
+		(drill 0.3)
+		(layers "F.Cu" "B.Cu")
+		(free yes)
+		(net "GND")
+	)
+	(via
 		(at 40.4495 129.159)
 		(size 0.6)
@@
 	)
 	(via
+		(at 49.6697 129.9972)
+		(size 0.6)
+		(drill 0.3)
+		(layers "F.Cu" "B.Cu")
+		(free yes)
+		(net "GND")
+	)
+	(via
 		(at 36.3065 119.7328)
 		(size 0.6)
@@
 	)
 	(via
+		(at 53.09605 136.347496)
+		(size 0.6)
+		(drill 0.3)
+		(layers "F.Cu" "B.Cu")
+		(free yes)
+		(net "GND")
+	)
+	(via
 		(at 72.6821 129.7686)
 		(size 0.6)
@@
 	)
 	(via
-		(at 39.3065 122.7328)
+		(at 49.6951 136.3726)
 		(size 0.6)
 		(drill 0.3)
 		(layers "F.Cu" "B.Cu")
+		(free yes)
 		(net "GND")
 	)
 	(via
-		(at 52.6987 121.4032)
+		(at 39.3065 122.7328)
 		(size 0.6)
 		(drill 0.3)
@@
 	)
 	(via
-		(at 69.7865 124.3866)
+		(at 52.6987 121.4032)
 		(size 0.6)
 		(drill 0.3)
@@
 	)
 	(via
-		(at 69.7865 127.3866)
+		(at 69.7865 124.3866)
 		(size 0.6)
 		(drill 0.3)
@@
 	)
 	(via
+		(at 54.8513 132.817187)
+		(size 0.6)
+		(drill 0.3)
+		(layers "F.Cu" "B.Cu")
+		(free yes)
+		(net "GND")
+	)
+	(via
+		(at 54.8513 131.678391)
+		(size 0.6)
+		(drill 0.3)
+		(layers "F.Cu" "B.Cu")
+		(free yes)
+		(net "GND")
+	)
+	(via
 		(at 52.6987 127.4032)
 		(size 0.6)
@@
 	)
 	(via
+		(at 54.8513 134.824754)
+		(size 0.6)
+		(drill 0.3)
+		(layers "F.Cu" "B.Cu")
+		(free yes)
+		(net "GND")
+	)
+	(via
 		(at 69.7357 143.9418)
 		(size 0.6)
@@
 	)
 	(via
+		(at 47.7647 129.9972)
+		(size 0.6)
+		(drill 0.3)
+		(layers "F.Cu" "B.Cu")
+		(free yes)
+		(net "GND")
+	)
+	(via
 		(at 38.3667 127.2794)
 		(size 0.6)
@@
 	)
 	(via
+		(at 54.8513 133.7564)
+		(size 0.6)
+		(drill 0.3)
+		(layers "F.Cu" "B.Cu")
+		(free yes)
+		(net "GND")
+	)
+	(via
 		(at 49.6987 124.4032)
 		(size 0.6)
@@
 		(polygon
 			(pts
-				(xy 44.9707 140.2842) (xy 61.8363 140.2842) (xy 61.8363 136.525) (xy 48.6283 136.525) (xy 48.6283 130.9116)
-				(xy 47.3075 130.9116) (xy 47.3075 136.6774) (xy 44.9707 136.6774)
+				(xy 44.9707 140.2842) (xy 61.8363 140.2842) (xy 61.8363 136.9822) (xy 48.6283 136.9822) (xy 48.6283 130.9116)
+				(xy 47.3075 130.9116) (xy 47.3075 136.9822) (xy 44.9707 136.9822)
 			)
 		)

Commit message: Add files via upload
Parts:
- removed the REF** at (27.1, 122.8)
- removed the REF** at (74.1, 146.7)
- removed the REF** at (27.1, 146.7)
- removed the REF** at (74.1, 122.8)
- added G***: LOGO, LOGO, F.Cu at (36.7, 122.8)
- added G***: LOGO, LOGO, B.Cu at (50.9, 137.7)
- added REF**: MountingHole_3.2mm_M3_Pad, MountingHole:MountingHole_3.2mm_M3_Pad, F.Cu at (74.8, 123.2)
- added REF**: MountingHole_3.2mm_M3_Pad, MountingHole:MountingHole_3.2mm_M3_Pad, F.Cu at (27.1, 123.2)
- added REF**: MountingHole_3.2mm_M3_Pad, MountingHole:MountingHole_3.2mm_M3_Pad, F.Cu at (27.1, 146.4)
- added REF**: MountingHole_3.2mm_M3_Pad, MountingHole:MountingHole_3.2mm_M3_Pad, F.Cu at (74.8, 146.4)
- moved C3 0.94 mm to (60.2, 143.8)
- moved C4 0.76 mm to (65.5, 142.2)
- moved J2 0.75 mm to (73.4, 135.6)
- moved J1 0.70 mm to (28.3, 132.1)
- moved L1 0.61 mm to (48.0, 144.0)
- moved C1 0.56 mm to (35.3, 139.9)
Routing:
- net GND: vias 50 -> 55
Other:
- board size 56.1 x 32.9 mm -> 56.8 x 32.8 mm
- board text added: "+ Input"
- board text added: "+ Output"
- board text added: "-"
- board text added: "- Input"
- board text added: "- Output"
- board text added: "GND"
- board text added: "Input"
- board text added: "Output"
- board text removed: "IN"
- board text removed: "LM2596-ADJ"
- board text removed: "OUT"
